Commit message: add palm camera. add callback for receiving images from the simple_run node

File: rbe4540-sim/ur_simulation_gz/ur_simulation_gz/urdf/ur_gz.urdf.xacro (robot description, xacro)
@@ -62,4 +62,70 @@
     <origin xyz="0 0 0.7" rpy="0 0 0" />          <!-- position robot in the world -->
   </xacro:ur_robot>
+  <!-- Palm camera: the gripper's +Z points out between the fingers.
+       Gazebo cameras look along +X, so rotate the camera link accordingly.
+       The housing starts at z = 107 mm; the lens is at 115 mm. -->
+  <joint name="$(arg tf_prefix)palm_camera_joint" type="fixed">
+    <parent link="$(arg tf_prefix)robotiq_robotiq_140_base_link"/>
+    <child link="$(arg tf_prefix)palm_camera_link"/>
+    <origin xyz="0 0 0.115" rpy="0 ${-pi/2} 0"/>
+  </joint>
+  <link name="$(arg tf_prefix)palm_camera_link">
+    <!-- Deliberately no collision geometry: the camera cannot contact the
+         object or fingers in Gazebo or introduce MoveIt collision checks. -->
+    <visual>
+      <origin xyz="-0.004 0 0" rpy="0 0 0"/>
+      <geometry>
+        <box size="0.008 0.018 0.018"/>
+      </geometry>
+      <material name="palm_camera_housing">
+        <color rgba="0.15 0.15 0.15 1"/>
+      </material>
+    </visual>
+    <visual>
+      <origin xyz="-0.0004 0 0" rpy="0 ${pi/2} 0"/>
+      <geometry>
+        <cylinder radius="0.004" length="0.001"/>
+      </geometry>
+      <material name="palm_camera_lens">
+        <color rgba="0.02 0.02 0.02 1"/>
+      </material>
+    </visual>
+    <inertial>
+      <origin xyz="-0.004 0 0" rpy="0 0 0"/>
+      <mass value="0.01"/>
+      <inertia ixx="0.00000054" ixy="0" ixz="0"
+               iyy="0.000000323333" iyz="0" izz="0.000000323333"/>
+    </inertial>
+  </link>
+  <!-- ROS optical convention: +Z forward, +X image right, +Y image down. -->
+  <joint name="$(arg tf_prefix)palm_camera_optical_joint" type="fixed">
+    <parent link="$(arg tf_prefix)palm_camera_link"/>
+    <child link="$(arg tf_prefix)palm_camera_optical_frame"/>
+    <origin xyz="0 0 0" rpy="${-pi/2} 0 ${-pi/2}"/>
+  </joint>
+  <link name="$(arg tf_prefix)palm_camera_optical_frame"/>
+  <gazebo reference="$(arg tf_prefix)palm_camera_link">
+    <sensor name="$(arg tf_prefix)palm_camera" type="camera">
+      <always_on>true</always_on>
+      <update_rate>30</update_rate>
+      <visualize>true</visualize>
+      <topic>/palm_camera/image</topic>
+      <gz_frame_id>$(arg tf_prefix)palm_camera_optical_frame</gz_frame_id>
+      <camera>
+        <camera_info_topic>/palm_camera/camera_info</camera_info_topic>
+        <optical_frame_id>$(arg tf_prefix)palm_camera_optical_frame</optical_frame_id>
+        <horizontal_fov>${pi/2}</horizontal_fov>
+        <image>
+          <width>640</width>
+          <height>480</height>
+          <format>R8G8B8</format>
+        </image>
+        <clip>
+          <near>0.001</near>
+          <far>5</far>
+        </clip>
+      </camera>
+    </sensor>
+  </gazebo>
   <gazebo reference="world">
   </gazebo>
